File: Current Sensor/Full (50A)/Current Sense.brd (EAGLE design)
At the start: 19.7 x 17.8 mm, 20 parts, among them IC1 INA169, IC2 REG1117

Commit message: Updated to V4.0
Parts:
- renumbered PAD1 to OUT, PAD3 to IN
Other:
- board text added: "+IN"
- board text added: "+OUT"
- board text added: "CC-BY-NC-SA"
- board text added: "Thayne Wade"
